File: POE-MicroMod-Function-Board.kicad_sch (KiCad schematic)
At the start: 0 parts

Commit message: started schematic
Parts:
- added C1: 10nF, symbol Device:C
- added C2: 4.7uF, symbol Device:C
- added R1: 12.4k, symbol Device:R
- added U1: W5500, Package_QFP:LQFP-48_7x7mm_P0.5mm, symbol Interface_Ethernet:W5500
Connections:
- new net: C1.1, U1.22 (1V2O)
- new net: R1.1, U1.10 (EXRES1)
- new net: U1.11 (AVDD), U1.15 (AVDD), U1.17 (AVDD), U1.21 (AVDD), U1.4 (AVDD), U1.8 (AVDD)
- new net: C2.1, U1.20 (TOCAP)
- new net ACTIVE_LED: U1.27 (ACTLED)
- new net CS: U1.32 (~{SCS})
- new net GND: C1.2, C2.2, R1.2, U1.14 (AGND), U1.16 (AGND), U1.19 (AGND), U1.29 (GND), U1.3 (AGND), U1.48 (AGND), U1.9 (AGND)
- new net INT: U1.36 (~{INT})
- new net LINK_LED: U1.25 (LINKLED)
- new net MISO: U1.34 (MISO)
- new net MOSI: U1.35 (MOSI)
- new net RST: U1.37 (~{RST})
- new net RX_N: U1.5 (RXN)
- new net RX_P: U1.6 (RXP)
- new net SCLK: U1.33 (SCLK)
- new net TX_N: U1.1 (TXN)
- new net TX_P: U1.2 (TXP)
- new net X_I: U1.30 (XI/CLKIN)
- new net X_O: U1.31 (XO)
- no-connect marks 0 -> 11

Commit message: updated libraries
Parts:
- added RJ1: HY931147C, HY931147C:RJ45-TH_HY931147C, symbol HY931147C:HY931147C
Changed lines of the file:
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@@
+	)
+	(symbol
+		(lib_id "HY931147C:HY931147C")
+		(at 224.79 50.8 0)
+		(unit 1)
+		(exclude_from_sim no)
+		(in_bom yes)
+		(on_board yes)
+		(dnp no)
+		(fields_autoplaced yes)
+		(property "Reference" "RJ1"
+			(at 260.35 49.5299 0)
+			(effects
+				(font
+					(size 1.27 1.27)
+				)
+				(justify left)
+			)
+		)
+		(property "Value" "HY931147C"
+			(at 260.35 52.0699 0)
+			(effects
+				(font
+					(size 1.27 1.27)
+				)
+				(justify left)
+			)
+		)
+		(property "Footprint" "HY931147C:RJ45-TH_HY931147C"
+			(at 224.79 50.8 0)
+			(effects
+				(font
+					(size 1.27 1.27)
+				)
+				(hide yes)
+			)
+		)
+		(property "Datasheet" ""
+			(at 224.79 50.8 0)
+			(effects
+				(font
+					(size 1.27 1.27)
+				)
+				(hide yes)
+			)
+		)
+		(property "Description" ""
+			(at 224.79 50.8 0)
+			(effects
+				(font
+					(size 1.27 1.27)
+				)
+				(hide yes)
+			)
+		)
+		(property "Manufacturer Part" "HY931147C"
+			(at 224.79 50.8 0)
+			(effects
+				(font
+					(size 1.27 1.27)
+				)
+				(hide yes)
+			)
+		)
+		(property "Manufacturer" "HANRUN(汉仁)"
+			(at 224.79 50.8 0)
+			(effects
+				(font
+					(size 1.27 1.27)
+				)
+				(hide yes)
+			)
+		)
+		(property "Supplier Part" "C91754"
+			(at 224.79 50.8 0)
+			(effects
+				(font
+					(size 1.27 1.27)
+				)
+				(hide yes)
+			)
+		)
+		(property "Supplier" "LCSC"
+			(at 224.79 50.8 0)
+			(effects
+				(font
+					(size 1.27 1.27)
+				)
+				(hide yes)
+			)
+		)
+		(pin "13"
+		)
+		(pin "14"
+		)
+		(pin "11"
+		)
+		(pin "12"
+		)
+		(pin "1"
+		)
+		(pin "9"
+		)
+		(pin "GND1"
+		)
+		(pin "GND2"
+		)
+		(pin "5"
+		)
+		(pin "10"
+		)
+		(pin "8"
+		)
+		(pin "7"
+		)
+		(pin "4"
+		)
+		(pin "6"
+		)
+		(pin "3"
+		)
+		(pin "2"
+		)
+		(instances
+			(project ""
+				(path "/38f6c0d4-acf1-4e69-be48-57e04aab2fd4"
+					(reference "RJ1")
+					(unit 1)
+				)
+			)
+		)
 	)
 	(symbol

Commit message: started routing pcb
Parts:
- removed RJ1: HY931147C, HY931147C:RJ45-TH_HY931147C, symbol HY931147C:HY931147C
- added C3: 10uF, symbol Device:C
- added C4: 100uF, symbol Device:C
- added C5, C6: 6.8n, Capacitor_SMD:C_0402_1005Metric, symbol Device:C
- added C7: 10n, Capacitor_SMD:C_0402_1005Metric, symbol Device:C
- added C8: 22u, Capacitor_SMD:C_0402_1005Metric, symbol Device:C
- added D1: SMAJ58A, Diode_SMD:D_SMA, symbol Diode:SMAJ58A
- added J1: ~, MicroMod:M.2-CARD-E-22_FUNCTION_STANDARD, symbol MicroMod:MICROMOD_FUNCTION_MAIN
- added R10, R4, R5, R8, R9: 49.9, Resistor_SMD:R_0402_1005Metric, symbol Device:R
- added R11, R12: 330, Resistor_SMD:R_0603_1608Metric, symbol Device:R
- added R2, R3, R6, R7: 33, Resistor_SMD:R_0402_1005Metric, symbol Device:R
- added RJ1: HY931147C, EasyEDA:RJ45-TH_HY931147C, symbol EasyEDA:HY931147C
- added U2: ~, EasyEDA:DM9900_5V, symbol EasyEDA:DM9900_5V
- C1, C2: footprint (none) -> Capacitor_SMD:C_0402_1005Metric
- R1: footprint (none) -> Resistor_SMD:R_0402_1005Metric
Connections:
- net ACTIVE_LED: now also R12.1
- net CS: now also J1.49 (F1/~{CS})
- net GND: now also C7.2, C8.2, J1.1 (GND), J1.2 (GND), J1.33 (GND), J1.39 (GND), J1.45 (GND), J1.75 (GND), J1.8 (GND), RJ1.10, RJ1.9, RJ1.GND1 (GND), RJ1.GND2 (GND)
- net INT: now also J1.47 (F0/~{INT})
- net LINK_LED: now also R11.2
- net MISO: now also J1.7 (SPI_SDO)
- net MOSI: now also J1.5 (SPI_SDI)
- net RST: now also J1.51 (F2/PWM)
- net RX_N: now also R2.1
- net RX_P: now also R3.1
- net SCLK: now also J1.3 (SPI_SCK)
- net TX_N: now also R6.1
- net TX_P: now also R7.1
- new net: C6.1, R3.2, R4.1
- new net: C7.1, R4.2, R5.2, RJ1.3
- new net: R7.2, R9.1, RJ1.5
- new net: C3.2, C4.2, U2.3 (VCC-)
- new net: C5.1, R2.2, R5.1
- new net: R6.2, R8.1, RJ1.6
- new net: R12.2, RJ1.13
- new net: C6.2, RJ1.1
- new net: R11.1, RJ1.11
- new net: C5.2, RJ1.2
- new net: C8.1, R10.1, RJ1.4
- new net: J1.72 (VCC), J1.74 (VCC)
- new net 3.3V: J1.73 (3.3V), R10.2, R8.2, R9.2, RJ1.12, RJ1.14
- new net 5V: C3.1, C4.1, U2.1 (VCC+), U2.2 (VCC+)
- new net POE+: D1.1 (A1), RJ1.7, U2.5 (VIN+), U2.6 (VIN+)
- new net POE-: D1.2 (A2), RJ1.8, U2.6 (VIN+), U2.7 (VIN-)
- no-connect marks 11 -> 43
Other:
- note added: "Capacitors should be 25V"
- note added: "https://docs.wiznet.io/assets/files/w5500_sch_v110_use_mag_-dfff8bbb103d13be4f25cd2b2f8b950d.pdf"
- moved on the sheet: C1, C2, R1, U1
